File: jammasplit.kicad_pcb (KiCad board)
At the start: 2 copper layers, 76.2 x 39.4 mm, 36 parts, among them J3 AV OUT, J4 AUDIO OUT, U1 THS7374

Commit message: v 0.1
v 0.1
Parts:
- removed C10, C12, C14, C2, C3, C4, C5, C8: 0.1uF, Capacitor_SMD:C_0805_2012Metric_Pad1.15x1.40mm_HandSolder
- removed C11, C13, C15, C9: 330uF, Capacitor_THT:CP_Radial_D6.3mm_P2.50mm
- removed R5, R6, R7, R8: 75, Resistor_SMD:R_0805_2012Metric_Pad1.15x1.40mm_HandSolder
- removed REF** (x4): MountingHole_2.5mm, MountingHole:MountingHole_2.5mm
- removed TY-145P: TY-145P, ty145p:TY-145P
- added ?: , MountingHole:MountingHole_2.5mm, F.Cu at (49.3, 110.5)
- added ?: , MountingHole:MountingHole_2.5mm, F.Cu at (49.3, 78.7)
- added ?: , MountingHole:MountingHole_2.5mm, F.Cu at (104.8, 110.5)
- added ?: , MountingHole:MountingHole_2.5mm, F.Cu at (104.8, 78.7)
- added CA: , Resistor_SMD:R_Array_Convex_4x0603, F.Cu at (71.1, 78.7)
- added JMP1: SCART_AUDIO, Resistor_SMD:R_0603_1608Metric_Pad1.05x0.95mm_HandSolder, B.Cu at (93.3, 94.6)
- added RA: , Resistor_SMD:R_Array_Convex_4x0603, F.Cu at (86.4, 78.7)
- added T1: TY-250P, SamacSys_Parts:TY250P, F.Cu at (87.7, 108.6)
- C7: value 0.1uF -> (none)
- J1: renamed from AV IN
- moved R1 22.2 mm to (76.2, 85.1), turned to 0 degrees
- moved R4 22.2 mm to (76.2, 88.9)
- moved C6 20.5 mm to (87.6, 87.6)
- moved J3 15.7 mm to (100.3, 97.8)
- moved J4 15.6 mm to (107.4, 86.4)
- moved R3 6.48 mm to (71.1, 85.1)
- moved R9 5.68 mm to (81.3, 85.1)
- moved D1 3.59 mm to (81.3, 88.9)
- moved R2 1.27 mm to (71.1, 88.9)
- moved C7 1.07 mm to (86.4, 82.5)
- moved U1 0.37 mm to (78.7, 80.6)
- renumbered BLUE1 to BLUE, GREEN1 to GREEN, RED1 to RED
Connections:
- J4 pad R: AUDIO_MONO_OUT -> Net-(J4-PadR)
- J4 pad T: AUDIO_MONO_OUT -> Net-(J4-PadR)
Routing:
- net AUDIO_MONO_OUT: track 56.1 -> 10.5 mm
- net Net-(J4-PadR): track 0.00 -> 34.3 mm
- net Net-(C14-Pad2): track 23.9 -> 0.00 mm
- net +AUDIO_IN: track 52.3 -> 31.4 mm, vias 1 -> 0
- net +5V: track 102.0 -> 83.0 mm, vias 1 -> 0
- net Net-(C12-Pad2): track 18.8 -> 0.00 mm
- net Net-(C10-Pad2): track 14.3 -> 0.00 mm
- net Net-(RA1-Pad4): track 16.8 -> 4.33 mm, vias 2 -> 0
- net Net-(C8-Pad2): track 12.2 -> 0.00 mm
- net BLUE_OUT: track 34.0 -> 23.3 mm, vias 0 -> 2
- net Net-(CA1-Pad8): track 13.8 -> 4.50 mm
- net Net-(R1-Pad2): track 15.9 -> 24.8 mm
- net Net-(CA1-Pad1): track 8.96 -> 17.1 mm, vias 0 -> 2
- net Net-(RA1-Pad3): track 12.2 -> 4.10 mm
- net GND: track 15.8 -> 9.07 mm, vias 2 -> 0
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Other:
- board size 76.2 x 39.4 mm -> 64.5 x 39.4 mm
- board text added: "+5V"
- board text added: "B"
- board text added: "G"
- board text added: "GND"
- board text added: "R"
- board text added: "S"
- board text added: "SP+"
- board text added: "SP-"
- board text added: "Ver 0.1"
- board text removed: "Ver 0.0"

Commit message: small fixes
Parts:
- renumbered RED to GREEN, GREEN to RED
Changed lines of the file:
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@@
   )
   (setup
-    (last_trace_width 0.5)
+    (last_trace_width 0.25)
     (user_trace_width 0.25)
     (user_trace_width 0.5)
@@
     (tags "resistor handsolder")
     (attr smd)
-    (fp_text reference JMP1 (at 0 1.905 270) (layer B.SilkS)
+    (fp_text reference JMP1 (at 0 1.905 270) (layer B.SilkS) hide
       (effects (font (size 1 1) (thickness 0.15)) (justify mirror))
     )
@@
     (descr "Potentiometer, vertical, Bourns 3386P, https://www.bourns.com/pdfs/3386.pdf")
     (tags "Potentiometer vertical Bourns 3386P")
-    (fp_text reference GREEN (at 5.871254 -2.523772 270) (layer F.SilkS)
+    (fp_text reference RED (at 5.871254 -2.523772 270) (layer F.SilkS)
       (effects (font (size 1 1) (thickness 0.15)))
     )
@@
     (descr "Potentiometer, vertical, Bourns 3386P, https://www.bourns.com/pdfs/3386.pdf")
     (tags "Potentiometer vertical Bourns 3386P")
-    (fp_text reference RED (at 5.838797 -2.593713 90) (layer F.SilkS)
+    (fp_text reference GREEN (at 5.838797 -2.593713 90) (layer F.SilkS)
       (effects (font (size 1 1) (thickness 0.15)))
     )
@@
     (tags "SSOP 0.65")
     (attr smd)
-    (fp_text reference U1 (at 0.010569 -1.553761) (layer F.SilkS) hide
+    (fp_text reference U1 (at 0 -0.060922) (layer F.SilkS)
       (effects (font (size 1 1) (thickness 0.15)))
     )
@@
     (fp_line (start 0.8 -1.6) (end 0.8 1.6) (layer F.Fab) (width 0.1))
     (fp_line (start -0.8 -1.6) (end 0.8 -1.6) (layer F.Fab) (width 0.1))
-    (fp_text user %R (at 0 0 90) (layer F.SilkS)
+    (fp_text user %R (at 0 0 90) (layer F.SilkS) hide
       (effects (font (size 0.5 0.5) (thickness 0.075)))
     )
@@
     (tags "resistor array")
     (attr smd)
-    (fp_text reference RA (at 0 -2.54) (layer F.SilkS) hide
+    (fp_text reference RA (at 0 -2.54) (layer F.SilkS)
       (effects (font (size 1 1) (thickness 0.15)))
     )
@@
       (effects (font (size 1 1) (thickness 0.15)))
     )
-    (fp_text user %R (at 0 0 90) (layer F.SilkS)
+    (fp_text user %R (at 0 0 90) (layer F.SilkS) hide
       (effects (font (size 0.5 0.5) (thickness 0.075)))
     )
@@
       (effects (font (size 1.27 1.27) (thickness 0.254)))
     )
-    (fp_text value TY-250P (at -6.604 -4.479001) (layer F.SilkS) hide
+    (fp_text value TY-250P (at -6.604 -4.479001) (layer F.SilkS)
       (effects (font (size 1.27 1.27) (thickness 0.254)))
     )
@@
   (gr_line (start 109.22 74.93) (end 109.22 114.3) (layer Edge.Cuts) (width 0.05))
   (gr_line (start 44.704 74.93) (end 109.22 74.93) (layer Edge.Cuts) (width 0.05))
-  (gr_text "BETSU\nBETSU" (at 97.00634 78.375068) (layer F.SilkS)
+  (gr_text "BETSU\nBETSU" (at 96.945714 78.638265) (layer F.SilkS)
     (effects (font (size 1.5 1.5) (thickness 0.3) italic))
   )

Commit message: Small fixes
Parts:
- removed ? (x4): , MountingHole:MountingHole_2.5mm
- added H1: MountingHole, MountingHole:MountingHole_2.5mm, F.Cu at (48.3, 110.5)
- added H2: MountingHole, MountingHole:MountingHole_2.5mm, F.Cu at (48.3, 79.2)
- added H3: MountingHole, MountingHole:MountingHole_2.5mm, F.Cu at (105.4, 78.7)
- added H4: MountingHole, MountingHole:MountingHole_2.5mm, F.Cu at (105.4, 110.5)
- C2: renamed from C7; value (none) -> 0.1uF
- CA1: renamed from CA; value (none) -> CapacitorArray4
- RA1: renamed from RA; value (none) -> ResistorArray4
- renumbered C6 to C1, J3 to J2, J4 to J3, R2 to R1, R3 to R2, R9 to R3, R1 to R4, R4 to R5, RED to RV1, GREEN to RV2, BLUE to RV3
